File: src/max1749-breakout.brd (EAGLE design)
At the start: 15.6 x 5.4 mm, 7 parts, among them J1 PTH VERT MALE, J2 PTH VERT MALE, U1 MAX1749EUK+T

Commit message: Update CAM files.
Other:
- board size 15.6 x 5.4 mm -> 15.6 x 6 mm
Changed lines of the file:
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@@
 <setting verticaltext="up"/>
 </settings>
-<grid distance="0.5" unitdist="mm" unit="mm" style="lines" multiple="1" display="yes" altdistance="0.1" altunitdist="mm" altunit="mm"/>
+<grid distance="0.3" unitdist="mm" unit="mm" style="lines" multiple="1" display="yes" altdistance="0.1" altunitdist="mm" altunit="mm"/>
 <layers>
 <layer number="1" name="Top" color="4" fill="1" visible="yes" active="yes"/>
@@
 <board>
 <plain>
-<wire x1="-7.8" y1="-2.7" x2="7.8" y2="-2.7" width="0" layer="20"/>
-<wire x1="7.8" y1="-2.7" x2="7.8" y2="2.7" width="0" layer="20"/>
-<wire x1="7.8" y1="2.7" x2="-7.8" y2="2.7" width="0" layer="20"/>
-<wire x1="-7.8" y1="2.7" x2="-7.8" y2="-2.7" width="0" layer="20"/>
+<wire x1="-7.8" y1="-3" x2="7.8" y2="-3" width="0" layer="20"/>
+<wire x1="7.8" y1="-3" x2="7.8" y2="3" width="0" layer="20"/>
+<wire x1="7.8" y1="3" x2="-7.8" y2="3" width="0" layer="20"/>
+<wire x1="-7.8" y1="3" x2="-7.8" y2="-3" width="0" layer="20"/>
 <text x="-4.5" y="1.27" size="0.5" layer="21" font="vector" ratio="10" align="center-left">ON</text>
 <text x="-4.5" y="-1.27" size="0.5" layer="21" font="vector" ratio="10" align="center-left">VIN</text>
@@
 </class>
 </classes>
-<designrules name="stella-wearables">
-<description language="en">&lt;b&gt;Stella Wearables Design Rules based on OSH Park Design Rules&lt;/b&gt;
+<designrules name="oshpark-2layer">
+<description language="en">&lt;b&gt;OSH Park Design Rules&lt;/b&gt;
 &lt;p&gt;
 Please make sure your boards conform to these design rules.
@@
 <param name="mtCopper" value="0.035559375mm 0.0356mm 0.0356mm 0.0356mm 0.0356mm 0.0356mm 0.0356mm 0.0356mm 0.0356mm 0.0356mm 0.0356mm 0.0356mm 0.0356mm 0.0356mm 0.0356mm 0.035559375mm"/>
 <param name="mtIsolate" value="1.6mm 0.1499mm 0.2007mm 0.1499mm 0.2007mm 0.1499mm 0.2007mm 0.1499mm 0.2007mm 0.1499mm 0.2007mm 0.1499mm 0.2007mm 0.1499mm 0.2007mm"/>
-<param name="mdWireWire" value="3mil"/>
-<param name="mdWirePad" value="3mil"/>
-<param name="mdWireVia" value="3mil"/>
-<param name="mdPadPad" value="3mil"/>
-<param name="mdPadVia" value="3mil"/>
-<param name="mdViaVia" value="3mil"/>
-<param name="mdSmdPad" value="3mil"/>
-<param name="mdSmdVia" value="3mil"/>
-<param name="mdSmdSmd" value="3mil"/>
+<param name="mdWireWire" value="6mil"/>
+<param name="mdWirePad" value="6mil"/>
+<param name="mdWireVia" value="6mil"/>
+<param name="mdPadPad" value="6mil"/>
+<param name="mdPadVia" value="6mil"/>
+<param name="mdViaVia" value="6mil"/>
+<param name="mdSmdPad" value="6mil"/>
+<param name="mdSmdVia" value="6mil"/>
+<param name="mdSmdSmd" value="6mil"/>
 <param name="mdViaViaSameLayer" value="8mil"/>
 <param name="mnLayersViaInSmd" value="2"/>
@@
 <param name="mdDrill" value="6mil"/>
 <param name="mdSmdStop" value="0mil"/>
-<param name="msWidth" value="3mil"/>
-<param name="msDrill" value="6mil"/>
+<param name="msWidth" value="6mil"/>
+<param name="msDrill" value="10mil"/>
 <param name="msMicroVia" value="10mil"/>
 <param name="msBlindViaRatio" value="0.5"/>
@@
 <signal name="VLED">
 <polygon width="0.1524" layer="16">
-<vertex x="-7.8" y="-2.7"/>
-<vertex x="7.8" y="-2.7"/>
-<vertex x="7.8" y="2.7"/>
-<vertex x="-7.8" y="2.7"/>
+<vertex x="-7.8" y="-3"/>
+<vertex x="7.8" y="-3"/>
+<vertex x="7.8" y="3"/>
+<vertex x="-7.8" y="3"/>
 </polygon>
 </signal>
@@
 <contactref element="J2" pad="1"/>
 <polygon width="0.1524" layer="1">
-<vertex x="-7.8" y="-2.7"/>
-<vertex x="7.8" y="-2.7"/>
-<vertex x="7.8" y="2.7"/>
-<vertex x="-7.8" y="2.7"/>
+<vertex x="-7.8" y="-3"/>
+<vertex x="7.8" y="-3"/>
+<vertex x="7.8" y="3"/>
+<vertex x="-7.8" y="3"/>
 </polygon>
 </signal>
